File: sensor-board/kicad/sensor-board/sensor-board.kicad_pcb (KiCad board)
At the start: 2 copper layers, 29.5 x 20.3 mm, 13 parts, among them J1 Conn_01x04_Female, J2 Conn_01x02_Female, J3 Conn_01x03_Female, J4 Conn_01x02_Female, U1 LM324, U2 ATtiny25-20SU

Commit message: Sensor-board: revize 2
Opravená chyba: Operační zesilovač má silnější výstup než programátor,
takže kompletně sestavená revize 1 nelze snadno flashnout.
Parts:
- added R7: 2k2, Resistor_SMD:R_1206_3216Metric_Pad1.42x1.75mm_HandSolder, B.Cu at (168.9, 66.0)
- R1, R2, R3, R4: value R -> 100R
- R5, R6: value R -> 16k
Connections:
- U1 pad 14: Net-(J4-Pad1) -> Net-(R7-Pad2)
Routing:
- net Net-(J4-Pad1): track 31.1 -> 27.4 mm, vias 0 -> 1
- net Net-(R7-Pad2): track 0.00 -> 2.32 mm
- net GND: vias 13 -> 12
Other:
- board text added: "Anemo Rev. 2"
- board text removed: "Anemo Rev. 1"
Changed lines of the file:
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@@
     (thickness 1.6)
     (drawings 21)
-    (tracks 114)
+    (tracks 115)
     (zones 0)
-    (modules 13)
-    (nets 14)
+    (modules 14)
+    (nets 15)
   )
   (page A4)
@@
   (net 12 "Net-(J1-Pad1)")
   (net 13 "Net-(J4-Pad1)")
+  (net 14 "Net-(R7-Pad2)")
   (net_class Default "This is the default net class."
     (clearance 0.2)
@@
     (add_net "Net-(R3-Pad2)")
     (add_net "Net-(R4-Pad2)")
+    (add_net "Net-(R7-Pad2)")
     (add_net "Net-(U1-Pad7)")
     (add_net "Net-(U1-Pad8)")
+  )
+  (module Resistor_SMD:R_1206_3216Metric_Pad1.42x1.75mm_HandSolder (layer B.Cu)
+    (at 168.91 66.04)
+    (descr "Resistor SMD 1206 (3216 Metric), square (rectangular) end terminal, IPC_7351 nominal with elongated pad for handsoldering. (Body size source: http://www.tortai-tech.com/upload/download/2011102023233369053.pdf), generated with kicad-footprint-generator")
+    (tags "resistor handsolder")
+    (attr smd)
+    (fp_text reference R7 (at 0 1.82) (layer B.SilkS)
+      (effects (font (size 1 1) (thickness 0.15)) (justify mirror))
+    )
+    (fp_text value 2k2 (at 0 -1.82) (layer B.Fab)
+      (effects (font (size 1 1) (thickness 0.15)) (justify mirror))
+    )
+    (fp_line (start -1.6 -0.8) (end -1.6 0.8) (layer B.Fab) (width 0.1))
+    (fp_line (start -1.6 0.8) (end 1.6 0.8) (layer B.Fab) (width 0.1))
+    (fp_line (start 1.6 0.8) (end 1.6 -0.8) (layer B.Fab) (width 0.1))
+    (fp_line (start 1.6 -0.8) (end -1.6 -0.8) (layer B.Fab) (width 0.1))
+    (fp_line (start -0.602064 0.91) (end 0.602064 0.91) (layer B.SilkS) (width 0.12))
+    (fp_line (start -0.602064 -0.91) (end 0.602064 -0.91) (layer B.SilkS) (width 0.12))
+    (fp_line (start -2.45 -1.12) (end -2.45 1.12) (layer B.CrtYd) (width 0.05))
+    (fp_line (start -2.45 1.12) (end 2.45 1.12) (layer B.CrtYd) (width 0.05))
+    (fp_line (start 2.45 1.12) (end 2.45 -1.12) (layer B.CrtYd) (width 0.05))
+    (fp_line (start 2.45 -1.12) (end -2.45 -1.12) (layer B.CrtYd) (width 0.05))
+    (fp_text user %R (at 0 0) (layer B.Fab)
+      (effects (font (size 0.8 0.8) (thickness 0.12)) (justify mirror))
+    )
+    (pad 1 smd roundrect (at -1.4875 0) (size 1.425 1.75) (layers B.Cu B.Paste B.Mask) (roundrect_rratio 0.175439)
+      (net 13 "Net-(J4-Pad1)"))
+    (pad 2 smd roundrect (at 1.4875 0) (size 1.425 1.75) (layers B.Cu B.Paste B.Mask) (roundrect_rratio 0.175439)
+      (net 14 "Net-(R7-Pad2)"))
+    (model ${KISYS3DMOD}/Resistor_SMD.3dshapes/R_1206_3216Metric.wrl
+      (at (xyz 0 0 0))
+      (scale (xyz 1 1 1))
+      (rotate (xyz 0 0 0))
+    )
   )
   (module Capacitor_THT:C_Radial_D5.0mm_H7.0mm_P2.00mm (layer F.Cu)
@@
       (net 11 "Net-(U1-Pad7)"))
     (pad 14 thru_hole oval (at 7.62 0) (size 1.6 1.6) (drill 0.8) (layers *.Cu *.Mask)
-      (net 13 "Net-(J4-Pad1)"))
+      (net 14 "Net-(R7-Pad2)"))
     (model ${KISYS3DMOD}/Package_DIP.3dshapes/DIP-14_W7.62mm.wrl
       (at (xyz 0 0 0))
@@
       (effects (font (size 1 1) (thickness 0.15)) (justify mirror))
     )
-    (fp_text value R (at 0 -1.82 270) (layer B.Fab)
+    (fp_text value 16k (at 0 -1.82 270) (layer B.Fab)
       (effects (font (size 1 1) (thickness 0.15)) (justify mirror))
     )
@@
       (effects (font (size 1 1) (thickness 0.15)) (justify mirror))
     )
-    (fp_text value R (at 0 -1.82 270) (layer B.Fab)
+    (fp_text value 16k (at 0 -1.82 270) (layer B.Fab)
       (effects (font (size 1 1) (thickness 0.15)) (justify mirror))
     )
@@
     (tags "resistor handsolder")
     (attr smd)
-    (fp_text reference R4 (at -3.81 0 270) (layer B.SilkS)
-      (effects (font (size 1 1) (thickness 0.15)) (justify mirror))
-    )
-    (fp_text value R (at 0 -1.82 270) (layer B.Fab)
+    (fp_text reference R4 (at -3.81 -0.508 270) (layer B.SilkS)
+      (effects (font (size 1 1) (thickness 0.15)) (justify mirror))
+    )
+    (fp_text value 100R (at 0 -1.82 270) (layer B.Fab)
       (effects (font (size 1 1) (thickness 0.15)) (justify mirror))
     )
@@
     (tags "resistor handsolder")
     (attr smd)
-    (fp_text reference R3 (at 3.81 0 90) (layer B.SilkS)
-      (effects (font (size 1 1) (thickness 0.15)) (justify mirror))
-    )
-    (fp_text value R (at 0 -1.82 90) (layer B.Fab)
+    (fp_text reference R3 (at 3.81 -0.508 90) (layer B.SilkS)
+      (effects (font (size 1 1) (thickness 0.15)) (justify mirror))
+    )
+    (fp_text value 100R (at 0 -1.82 90) (layer B.Fab)
       (effects (font (size 1 1) (thickness 0.15)) (justify mirror))
     )
@@
       (effects (font (size 1 1) (thickness 0.15)) (justify mirror))
     )
-    (fp_text value R (at 0 -1.82 90) (layer B.Fab)
+    (fp_text value 100R (at 0 -1.82 90) (layer B.Fab)
       (effects (font (size 1 1) (thickness 0.15)) (justify mirror))
     )
@@
       (effects (font (size 1 1) (thickness 0.15)) (justify mirror))
     )
-    (fp_text value R (at 0 -1.82 90) (layer B.Fab)
+    (fp_text value 100R (at 0 -1.82 90) (layer B.Fab)
       (effects (font (size 1 1) (thickness 0.15)) (justify mirror))
     )
@@
     )
   )
-  (gr_text "Anemo\nRev. 1" (at 158.115 68.58 90) (layer B.SilkS)
+  (gr_text "Anemo\nRev. 2" (at 158.115 68.58 90) (layer B.SilkS)
     (effects (font (size 1 1) (thickness 0.15)) (justify left mirror))
   )
@@
   (via (at 175.26 66.04) (size 0.8) (drill 0.4) (layers F.Cu B.Cu) (net 3))
   (via (at 160.02 75.565) (size 0.8) (drill 0.4) (layers F.Cu B.Cu) (net 3))
-  (via (at 167.64 65.405) (size 0.8) (drill 0.4) (layers F.Cu B.Cu) (net 3))
   (via (at 174.625 81.28) (size 0.8) (drill 0.4) (layers F.Cu B.Cu) (net 3))
   (via (at 178.435 69.215) (size 0.8) (drill 0.4) (layers F.Cu B.Cu) (net 3))
@@
   (segment (start 163.576 71.628) (end 163.576 68.072) (width 0.25) (layer F.Cu) (net 13))
   (segment (start 163.576 68.072) (end 156.464 68.072) (width 0.25) (layer F.Cu) (net 13))
-  (segment (start 163.576 68.072) (end 164.338 67.31) (width 0.25) (layer F.Cu) (net 13))
-  (segment (start 168.91 66.04) (end 172.72 66.04) (width 0.25) (layer F.Cu) (net 13))
-  (segment (start 167.64 67.31) (end 168.91 66.04) (width 0.25) (layer F.Cu) (net 13))
-  (segment (start 164.338 67.31) (end 167.64 67.31) (width 0.25) (layer F.Cu) (net 13))
   (segment (start 162.941 72.771) (end 160.655 72.771) (width 0.25) (layer F.Cu) (net 13))
+  (via (at 167.4225 67.945) (size 0.8) (drill 0.4) (layers F.Cu B.Cu) (net 13))
+  (segment (start 164.338 67.31) (end 163.576 68.072) (width 0.25) (layer F.Cu) (net 13))
+  (segment (start 166.7875 67.31) (end 167.4225 67.945) (width 0.25) (layer F.Cu) (net 13))
+  (segment (start 164.338 67.31) (end 166.7875 67.31) (width 0.25) (layer F.Cu) (net 13))
+  (segment (start 167.4225 66.04) (end 167.4225 67.945) (width 0.25) (layer B.Cu) (net 13))
+  (segment (start 170.3975 66.04) (end 172.72 66.04) (width 0.25) (layer B.Cu) (net 14))
   (zone (net 3) (net_name GND) (layer F.Cu) (hatch edge 0.508)
     (connect_pads (clearance 0.508))
